File: PTP1_LV.kicad_sch (KiCad schematic)
At the start: 0 parts

Commit message: ispunjena sastavnica
Parts:
- added R1, R2: R_Small, symbol Device:R_Small
Connections:
- new net +3V3: R2.1
- new net GND: R1.2
- new net U_izl: R1.1, R2.2
Other:
- company: (none) -> TVZ - tehničko veleučilište u Zagrebu
- title: (none) -> BCD brojač
